Commit message: Ros2 control tag for ethercat

File: esn_description/urdf/esn_ros2_control.xacro (robot description, xacro)
@@ -4,5 +4,22 @@
     <ros2_control name="${name}" type="system">
       <hardware>
-        <!-- Caso in simulazione -->
+        <!-- A prescindere questo giunto è simulato -->
+        <plugin>mock_components/GenericSystem</plugin>
+        <param name="mock_sensor_commands">true</param>
+        <joint name="${prefix}wheel_left_joint">
+          <command_interface name="position"/>
+          <command_interface name="velocity"/>
+          <state_interface name="position">
+            <param name="initial_value">0.0</param>
+          </state_interface>
+          <state_interface name="velocity">
+            <param name="initial_value">0.0</param>
+          </state_interface>
+          <state_interface name="effort">
+            <param name="initial_value">0.0</param>
+          </state_interface>
+        </joint>
+      </hardware>
+      <hardware>
         <xacro:if value="${use_fake_hardware}">
           <plugin>mock_components/GenericSystem</plugin>
@@ -10,23 +27,10 @@
         </xacro:if>
         <!-- Caso con hardware reale: ETHERCAT -->
-        <!-- <xacro:unless value="${use_fake_hardware}">
+        <xacro:unless value="${use_fake_hardware}">
           <plugin>ethercat_driver/EthercatDriver</plugin>
           <param name="master_id">${master_id}</param>
           <param name="control_frequency">1000</param>
-        </xacro:unless> -->
+        </xacro:unless>
       </hardware>
-      <joint name="${prefix}wheel_left_joint">
-        <command_interface name="position"/>
-        <command_interface name="velocity"/>
-        <state_interface name="position">
-          <param name="initial_value">0.0</param>
-        </state_interface>
-        <state_interface name="velocity">
-          <param name="initial_value">0.0</param>
-        </state_interface>
-        <state_interface name="effort">
-          <param name="initial_value">0.0</param>
-        </state_interface>
-      </joint>
       <joint name="${prefix}wheel_right_joint">
         <command_interface name="position"/>
@@ -41,4 +45,10 @@
           <param name="initial_value">0.0</param>
         </state_interface>
+        <ec_module name="${prefix}wheel_right_joint">
+          <plugin>ethercat_generic_plugins/GenericEcSlave</plugin>
+          <param name="alias">0</param>
+          <param name="position">0</param>
+          <param name="slave_config">$(find esn_description)/config/el7211_config.yaml</param>
+        </ec_module>
       </joint>
     </ros2_control>

Commit message: wip

File: esn_description/urdf/esn_ros2_control.xacro (robot description, xacro)
@@ -2,5 +2,5 @@
 <robot xmlns:xacro="http://www.ros.org/wiki/xacro">
   <xacro:macro name="esn_ros2_control" params="use_fake_hardware:=true name:=esn_robot prefix:=''">
-    <ros2_control name="${name}" type="system">
+    <ros2_control name="${name}_left" type="system">
       <hardware>
         <!-- A prescindere questo giunto è simulato -->
@@ -21,4 +21,6 @@
         </joint>
       </hardware>
+    </ros2_control>
+    <ros2_control name="${name}_right" type="system">
       <hardware>
         <xacro:if value="${use_fake_hardware}">
@@ -32,24 +34,27 @@
           <param name="control_frequency">1000</param>
         </xacro:unless>
+        <joint name="${prefix}wheel_right_joint">
+          <command_interface name="position"/>
+          <command_interface name="velocity"/>
+          <state_interface name="position">
+            <param name="initial_value">0.0</param>
+          </state_interface>
+          <state_interface name="velocity">
+            <param name="initial_value">0.0</param>
+          </state_interface>
+          <state_interface name="effort">
+            <param name="initial_value">0.0</param>
+          </state_interface>
+          <xacro:unless value="${use_fake_hardware}">
+            <ec_module name="${prefix}wheel_right_joint">
+              <plugin>ethercat_generic_plugins/EcCiA402Drive</plugin>
+              <param name="alias">0</param>
+              <param name="position">0</param>
+              <param name="mode_of_operation">9</param>
+              <param name="slave_config">$(find esn_description)/config/el7211_config.yaml</param>
+            </ec_module>
+          </xacro:unless>
+        </joint>
       </hardware>
-      <joint name="${prefix}wheel_right_joint">
-        <command_interface name="position"/>
-        <command_interface name="velocity"/>
-        <state_interface name="position">
-          <param name="initial_value">0.0</param>
-        </state_interface>
-        <state_interface name="velocity">
-          <param name="initial_value">0.0</param>
-        </state_interface>
-        <state_interface name="effort">
-          <param name="initial_value">0.0</param>
-        </state_interface>
-        <ec_module name="${prefix}wheel_right_joint">
-          <plugin>ethercat_generic_plugins/GenericEcSlave</plugin>
-          <param name="alias">0</param>
-          <param name="position">0</param>
-          <param name="slave_config">$(find esn_description)/config/el7211_config.yaml</param>
-        </ec_module>
-      </joint>
     </ros2_control>
   </xacro:macro>

Commit message: Ethercat ros2 tag ok

File: esn_description/urdf/esn_ros2_control.xacro (robot description, xacro)
@@ -1,5 +1,5 @@
 <?xml version="1.0"?>
 <robot xmlns:xacro="http://www.ros.org/wiki/xacro">
-  <xacro:macro name="esn_ros2_control" params="use_fake_hardware:=true name:=esn_robot prefix:=''">
+  <xacro:macro name="esn_ros2_control" params="use_fake_hardware:=true name:=esn_robot prefix:='' master_id:=0">
     <ros2_control name="${name}_left" type="system">
       <hardware>
@@ -7,18 +7,18 @@
         <plugin>mock_components/GenericSystem</plugin>
         <param name="mock_sensor_commands">true</param>
-        <joint name="${prefix}wheel_left_joint">
-          <command_interface name="position"/>
-          <command_interface name="velocity"/>
-          <state_interface name="position">
-            <param name="initial_value">0.0</param>
-          </state_interface>
-          <state_interface name="velocity">
-            <param name="initial_value">0.0</param>
-          </state_interface>
-          <state_interface name="effort">
-            <param name="initial_value">0.0</param>
-          </state_interface>
-        </joint>
       </hardware>
+      <joint name="${prefix}wheel_left_joint">
+        <command_interface name="position"/>
+        <command_interface name="velocity"/>
+        <state_interface name="position">
+          <param name="initial_value">0.0</param>
+        </state_interface>
+        <state_interface name="velocity">
+          <param name="initial_value">0.0</param>
+        </state_interface>
+        <state_interface name="effort">
+          <param name="initial_value">0.0</param>
+        </state_interface>
+      </joint>
     </ros2_control>
     <ros2_control name="${name}_right" type="system">
@@ -34,4 +34,5 @@
           <param name="control_frequency">1000</param>
         </xacro:unless>
+      </hardware>
         <joint name="${prefix}wheel_right_joint">
           <command_interface name="position"/>
@@ -56,5 +57,4 @@
           </xacro:unless>
         </joint>
-      </hardware>
     </ros2_control>
   </xacro:macro>
